File: board/bubblebutbot/bubblebutbot.kicad_sch (KiCad schematic)
At the start: 45 parts, among them J1 JST XH, J10 JST XH, J11 JST XH, J12 JST XH, J2 USB_C_Receptacle, J3 Conn_01x03_Socket, J4 Conn_01x03_Socket, J5 Conn_01x03_Socket, J6 Conn_01x03_Socket, J7 Conn_01x03_Socket, J8 Conn_01x03_Socket, J9 JST XH, Q1 FDN336P, SW1 SW_SPST, SW2 SW_SPST, SW3 SW_DIP_x04, U1 DRV8833PWP, U2 ESP32-S3-WROOM-1, U3 AP2112K-3.3, U4 LIS3DH

Commit message: added buck to 5V
Parts:
- added C11: 100n, Capacitor_SMD:C_0603_1608Metric_Pad1.08x0.95mm_HandSolder, symbol Device:C
- added C12: 22u, symbol Device:C
- added C9: 10u, Capacitor_SMD:C_0603_1608Metric_Pad1.08x0.95mm_HandSolder, symbol Device:C
- added L1: 4.7u, symbol Device:L
- added R12: 5.1K, Resistor_SMD:R_0603_1608Metric_Pad0.98x0.95mm_HandSolder, symbol Device:R
- added R13: 5.1K, symbol Device:R
- added R14, R15: 100k, Resistor_SMD:R_0603_1608Metric_Pad0.98x0.95mm_HandSolder, symbol Device:R
- added R16: R, symbol Device:R
- added U5: ~, symbol CustomSymbols:SY8303
- R10: value 10k -> 5.1K
- R9: value 10k -> 5.1K; footprint (none) -> Resistor_SMD:R_0603_1608Metric_Pad0.98x0.95mm_HandSolder
Connections:
- net +7.5V: now also C9.1, R13.2, U5.5 (IN)
- net 3V_SUPPLY: now also R12.2; no longer R10.2
- net 5V_SUPPLY: now also R8.2, U3.3 (EN)
- net 5V_USB_POWER: now also R10.2
- net ESP32-ACC-INT1: now also U2.24 (GPIO47/SPICLK_P/SUBSPICLK_P_DIFF); no longer U2.19 (GPIO11/TOUCH11/ADC2_CH0/FSPID/FSPIIO5/SUBSPID)
- net ESP32-ACC-INT2: now also U2.25 (GPIO48/SPICLK_N/SUBSPICLK_N_DIFF); no longer U2.20 (GPIO12/TOUCH12/ADC2_CH1/FSPICLK/FSPIIO6/SUBSPICLK)
- net ESP32-ACC-SDA: now also R12.1; no longer R10.1
- net ESP32-IR-BL: now also U2.6 (GPIO6/TOUCH6/ADC1_CH5)
- net ESP32-IR-BR: now also U2.7 (GPIO7/TOUCH7/ADC1_CH6)
- net ESP32-IR-FL: now also U2.4 (GPIO4/TOUCH4/ADC1_CH3)
- net ESP32-IR-FR: now also U2.5 (GPIO5/TOUCH5/ADC1_CH4)
- net ESP32-MANUAL-AUTO: now also U2.20 (GPIO12/TOUCH12/ADC2_CH1/FSPICLK/FSPIIO6/SUBSPICLK); no longer U2.17 (GPIO9/TOUCH9/ADC1_CH8/FSPIHD/SUBSPIHD)
- net ESP32-OP-LED: now also U2.18 (GPIO10/TOUCH10/ADC1_CH9/FSPICS0/FSPIIO4/SUBSPICS0); no longer U2.21 (GPIO13/TOUCH13/ADC2_CH2/FSPIQ/FSPIIO7/SUBSPIQ)
- net ESP32-SERVO-EN: now also U2.21 (GPIO13/TOUCH13/ADC2_CH2/FSPIQ/FSPIIO7/SUBSPIQ); no longer U2.18 (GPIO10/TOUCH10/ADC1_CH9/FSPICS0/FSPIIO4/SUBSPICS0)
- net ESP32-SRV-B: now also U2.17 (GPIO9/TOUCH9/ADC1_CH8/FSPIHD/SUBSPIHD)
- net ESP32-SRV-F: now also U2.12 (GPIO8/TOUCH8/ADC1_CH7/SUBSPICS1)
- net ESP32-WIFI-ANALOG: now also U2.19 (GPIO11/TOUCH11/ADC2_CH0/FSPID/FSPIIO5/SUBSPID); no longer U2.12 (GPIO8/TOUCH8/ADC1_CH7/SUBSPICS1)
- net GND: now also R10.1, C12.2, R14.1, R16.2, U5.3 (GND), U5.4 (GND)
- net 5V_BAT: now reaches Q1.2 (S)
- net 5V_BAT: now also C12.1, L1.2, R15.2
- new net: R15.1, R16.1, U5.1 (FB)
- new net: R14.2, U5.2 (FS)
- new net: C11.1, U5.7 (BS)
- new net: C11.2, L1.1, U5.6 (LX)
- new net: C9.2, R13.1, U5.8 (EN)
Other:
- note added: "Cin: 4.7uF, Cbs: 10nF, L: 15uH, Cout: 22uF + 10uF, Rfs: 100k L: 4.7uH R2: 13.6K R1: 100k"
- note added: "Falta aacabar aqi! Procurar os proximos componentes!"
- moved on the sheet: C4, C5, D2, Q1, R8, U3

Commit message: finished schematic and BOM. Design is ready to start!
Parts:
- removed J12: JST XH, symbol Connector:Conn_01x02_Socket
- removed SW1, SW2: SW_SPST, symbol Switch:SW_SPST
- added D3: LED, LED_SMD:LED_0603_1608Metric_Pad1.05x0.95mm_HandSolder, symbol Device:LED
- added J13: JST XH, Connector_JST:JST_PH_S2B-PH-K_1x02_P2.00mm_Horizontal, symbol Connector:Conn_01x02_Socket
- added R17: 5.1K, Resistor_SMD:R_0603_1608Metric_Pad0.98x0.95mm_HandSolder, symbol Device:R
- added SW1, SW2: SW_Push, Button_Switch_SMD:SW_SPST_B3U-1000P, symbol Switch:SW_Push
- C12: footprint (none) -> Capacitor_SMD:C_1206_3216Metric_Pad1.33x1.80mm_HandSolder; LCSC (none) -> C12891
- C4, C5: footprint (none) -> Capacitor_SMD:C_0603_1608Metric_Pad1.08x0.95mm_HandSolder
- J1, J10, J11, J9: footprint (none) -> Connector_JST:JST_PH_S2B-PH-K_1x02_P2.00mm_Horizontal; LCSC C33132 -> C722769
- J3, J4, J5, J6, J7, J8: footprint (none) -> Connector_JST:JST_PH_S3B-PH-K_1x03_P2.00mm_Horizontal
- L1: footprint (none) -> Inductor_SMD:L_Wuerth_WE-TPC-3816; LCSC (none) -> C2879693
- R10, R13, R4, R6, R7: footprint (none) -> Resistor_SMD:R_0603_1608Metric_Pad0.98x0.95mm_HandSolder
- R16: footprint (none) -> Resistor_SMD:R_0603_1608Metric_Pad0.98x0.95mm_HandSolder; LCSC (none) -> C2930064
- U2: footprint Espressif:ESP32-S3-WROOM-1 -> RF_Module:ESP32-S3-WROOM-1
- U5: footprint (none) -> Package_TO_SOT_SMD:SOT-23-8; LCSC (none) -> C2937216
Connections:
- net 3V_SUPPLY is gone; now on net +3.3V: C10.1, C4.1, C6.1, R12.2, R9.2, U3.5 (VOUT), U4.1 (VDD_IO), U4.14 (VDD)
- net 5V_SUPPLY: no longer C5.1, D2.1 (K), J3.3 (Pin_3), J4.3 (Pin_3), J5.3 (Pin_3), J6.3 (Pin_3), J7.3 (Pin_3), J8.3 (Pin_3), Q1.3 (D), R8.1, R8.2, U3.1 (VIN), U3.3 (EN)
- net 5V_USB_POWER: now also R17.2
- net ESP32-BOOT0: now also SW2.1
- net ESP32-RESET: now also SW1.1
- net GND: now also D3.1 (K), SW1.2, SW2.2
- net MOTOR-LEFT-BL: now also J11.1 (Pin_1); no longer J9.1 (Pin_1)
- net MOTOR-LEFT-BR: now also J11.2 (Pin_2); no longer J9.2 (Pin_2)
- net MOTOR-RIGHT-BL: now also J9.1 (Pin_1), J13.1 (Pin_1); no longer J11.1 (Pin_1)
- net MOTOR-RIGHT-BR: now also J9.2 (Pin_2), J13.2 (Pin_2); no longer J11.2 (Pin_2)
- new net: D3.2 (A), R17.1
- new net +5V: C5.1, D2.1 (K), J3.3 (Pin_3), J4.3 (Pin_3), J5.3 (Pin_3), J6.3 (Pin_3), J7.3 (Pin_3), J8.3 (Pin_3), Q1.3 (D), R8.1, R8.2, U3.1 (VIN), U3.3 (EN)
Other:
- note removed: "5V BUCK: https://datasheet.lcsc.com/lcsc/1811151653_Silergy-Corp-SY8303AIC_C97054.pdf"
- note removed: "Falta aacabar aqi! Procurar os proximos componentes!"
- title: BubbleButBot Dev Board -> BubbleButBot Board
- moved on the sheet: C11, C12, C9, L1, R13, R14, R15, R16, U5

Commit message: a few more improvements here and there. Almost there.
Parts:
- removed R3: 5.1K, Resistor_SMD:R_0603_1608Metric_Pad0.98x0.95mm_HandSolder, symbol Device:R
- removed SW3: SW_DIP_x04, Button_Switch_THT:SW_DIP_SPSTx04_Piano_10.8x11.72mm_W7.62mm_P2.54mm, symbol Switch:SW_DIP_x04
Connections:
- net ESP32-MANUAL-AUTO is gone; now on net ESP32-ACC-SDA: U2.20 (GPIO12/TOUCH12/ADC2_CH1/FSPICLK/FSPIIO6/SUBSPICLK)
- net ESP32-SERVO-EN is gone; now on net ESP32-ACC-SCL: U2.21 (GPIO13/TOUCH13/ADC2_CH2/FSPIQ/FSPIIO7/SUBSPIQ)
- net ESP32-WIFI-ANALOG is gone; now on net ESP32-OP-LED: U2.19 (GPIO11/TOUCH11/ADC2_CH0/FSPID/FSPIIO5/SUBSPID)
- net +5V: no longer R8.2, U3.3 (EN)
- net ESP32-OP-LED: no longer U2.18 (GPIO10/TOUCH10/ADC1_CH9/FSPICS0/FSPIIO4/SUBSPICS0)
- net ESP32-SRV-F: now also U2.18 (GPIO10/TOUCH10/ADC1_CH9/FSPICS0/FSPIIO4/SUBSPICS0); no longer U2.12 (GPIO8/TOUCH8/ADC1_CH7/SUBSPICS1)
- new net: R8.2, U3.3 (EN)
Other:
- note removed: "Requires a pull-down resistor to be set on firmware!"
