File: board/bubblebutbot/bubblebutbot.kicad_sch (KiCad schematic)
At the start: 46 parts, among them J1 JST XH, J10 JST XH, J13 JST XH, J2 USB_C_Receptacle, J3 Conn_01x03_Socket, J4 Conn_01x03_Socket, J5 Conn_01x01_Pin, J6 Conn_01x01_Pin, J7 Conn_01x03_Socket, SW1 SW_Push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

Commit message: Working on the new version ... 🚀
Connections:
- net +3.3V: now also C4.1, C5.1, J3.3 (Pin_3), J4.3 (Pin_3), L1.2, U3.1 (FB)
- net BAT_OUT: now also J7.2 (Pin_2)
- removed net +5V: J3.3 (Pin_3), J4.3 (Pin_3), J7.2 (Pin_2)
Changed lines of the file:
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@@
   (title_block
     (title "BubbleButBot Board")
-    (date "2024-01-24")
+    (date "2024-01-25")
     (rev "2.06")
     (comment 1 "2.01: Added debounce C for Boot and Reset button")
@@
   (junction (at 312.42 115.57) (diameter 0) (color 0 0 0 0)
   )
-  (junction (at 312.42 37.465) (diameter 0) (color 0 0 0 0)
-  )
   (junction (at 127 138.43) (diameter 0) (color 0 0 0 0)
   )
@@
   (junction (at 90.17 36.195) (diameter 0) (color 0 0 0 0)
   )
-  (junction (at 199.39 70.485) (diameter 0) (color 0 0 0 0)
-  )
   (junction (at 301.625 37.465) (diameter 0) (color 0 0 0 0)
   )
+  (junction (at 199.39 70.485) (diameter 0) (color 0 0 0 0)
+  )
   (junction (at 134.62 157.48) (diameter 0) (color 0 0 0 0)
   )
@@
   (junction (at 276.86 115.57) (diameter 0) (color 0 0 0 0)
   )
+  (junction (at 322.58 102.235) (diameter 0) (color 0 0 0 0)
+  )
   (junction (at 90.17 23.495) (diameter 0) (color 0 0 0 0)
   )
@@
     (stroke (width 0) (type default))
   )
-  (wire (pts (xy 312.42 37.465) (xy 301.625 37.465))
-    (stroke (width 0) (type default))
-  )
   (polyline (pts (xy 201.93 84.455) (xy 274.32 84.455))
     (stroke (width 0) (type default))
@@
     (stroke (width 0) (type default))
   )
+  (wire (pts (xy 298.45 37.465) (xy 301.625 37.465))
+    (stroke (width 0) (type default))
+  )
   (wire (pts (xy 134.62 157.48) (xy 137.795 157.48))
     (stroke (width 0) (type default))
@@
     (stroke (width 0) (type default))
   )
-  (wire (pts (xy 312.42 37.465) (xy 353.695 37.465))
-    (stroke (width 0) (type default))
-  )
   (wire (pts (xy 301.625 161.925) (xy 309.88 161.925))
     (stroke (width 0) (type default))
@@
     (stroke (width 0) (type default))
   )
-  (wire (pts (xy 353.695 37.465) (xy 353.695 41.275))
+  (wire (pts (xy 353.695 36.195) (xy 353.695 41.275))
     (stroke (width 0) (type default))
   )
@@
     (stroke (width 0) (type default))
   )
+  (wire (pts (xy 301.625 37.465) (xy 312.42 37.465))
+    (stroke (width 0) (type default))
+  )
   (wire (pts (xy 168.275 170.18) (xy 191.135 170.18))
     (stroke (width 0) (type default))
@@
     (stroke (width 0) (type default))
   )
-  (wire (pts (xy 297.18 37.465) (xy 301.625 37.465))
-    (stroke (width 0) (type default))
-  )
   (wire (pts (xy 66.675 138.43) (xy 66.675 147.32))
     (stroke (width 0) (type default))
@@
     )
   )
+  (global_label "BAT_OUT" (shape input) (at 353.695 36.195 90) (fields_autoplaced)
+    (effects (font (size 1.27 1.27)) (justify left))
+    (property "Intersheetrefs" "${INTERSHEET_REFS}" (at 353.695 25.2874 90)
+      (effects (font (size 1.27 1.27)) (justify left) hide)
+    )
+  )
   (global_label "BAT_IN" (shape output) (at 362.585 154.94 0) (fields_autoplaced)
     (effects (font (size 1.27 1.27)) (justify left))
@@
     )
   )
-  (symbol (lib_id "power:+5V") (at 297.18 37.465 90) (unit 1)
-    (in_bom yes) (on_board yes) (dnp no) (fields_autoplaced)
-    (property "Reference" "#PWR033" (at 300.99 37.465 0)
-      (effects (font (size 1.27 1.27)) hide)
-    )
-    (property "Value" "+5V" (at 294.0051 37.465 90)
-      (effects (font (size 1.27 1.27)) (justify left))
-    )
-    (property "Footprint" "" (at 297.18 37.465 0)
-      (effects (font (size 1.27 1.27)) hide)
-    )
-    (property "Datasheet" "" (at 297.18 37.465 0)
-      (effects (font (size 1.27 1.27)) hide)
-    )
-    (pin "1")
-    (instances
-      (project "bubblebutbot"
-        (path "/2cd1342d-9ef7-44f7-8a7d-ec49b5dc5750"
-          (reference "#PWR033") (unit 1)
-        )
-      )
-    )
-  )
   (symbol (lib_id "Device:R") (at 205.105 61.595 270) (unit 1)
     (in_bom yes) (on_board yes) (dnp no)
@@
     )
   )
+  (symbol (lib_id "power:+3.3V") (at 322.58 102.235 0) (unit 1)
+    (in_bom yes) (on_board yes) (dnp no) (fields_autoplaced)
+    (property "Reference" "#PWR014" (at 322.58 106.045 0)
+      (effects (font (size 1.27 1.27)) hide)
+    )
+    (property "Value" "+3.3V" (at 322.58 98.1019 0)
+      (effects (font (size 1.27 1.27)))
+    )
+    (property "Footprint" "" (at 322.58 102.235 0)
+      (effects (font (size 1.27 1.27)) hide)
+    )
+    (property "Datasheet" "" (at 322.58 102.235 0)
+      (effects (font (size 1.27 1.27)) hide)
+    )
+    (pin "1")
+    (instances
+      (project "bubblebutbot"
+        (path "/2cd1342d-9ef7-44f7-8a7d-ec49b5dc5750"
+          (reference "#PWR014") (unit 1)
+        )
+      )
+    )
+  )
   (symbol (lib_id "Device:R") (at 45.085 148.59 180) (unit 1)
     (in_bom yes) (on_board yes) (dnp no) (fields_autoplaced)
@@
         )
       )
+    )
+  )
+  (symbol (lib_id "power:+3.3V") (at 298.45 37.465 90) (unit 1)
+    (in_bom yes) (on_board yes) (dnp no) (fields_autoplaced)
+    (property "Reference" "#PWR020" (at 302.26 37.465 0)
+      (effects (font (size 1.27 1.27)) hide)
+    )
+    (property "Value" "+3.3V" (at 295.275 37.465 90)
+      (effects (font (size 1.27 1.27)) (justify left))
+    )
+    (property "Footprint" "" (at 298.45 37.465 0)
+      (effects (font (size 1.27 1.27)) hide)
+    )
+    (property "Datasheet" "" (at 298.45 37.465 0)
+      (effects (font (size 1.27 1.27)) hide)
+    )
+    (pin "1")
+    (instances
+      (project "bubblebutbot"
+        (path "/2cd1342d-9ef7-44f7-8a7d-ec49b5dc5750"
+          (reference "#PWR020") (unit 1)
+        )
+      )

Commit message: VERSION 1.06
Parts:
- removed C16: 22u, Capacitor_SMD:C_1206_3216Metric_Pad1.33x1.80mm_HandSolder, symbol Device:C
- removed J5, J6: Conn_01x01_Pin, TestPoint:TestPoint_Pad_2.0x2.0mm, symbol Connector:Conn_01x01_Pin
- L1: footprint Inductor_SMD:L_Wuerth_WE-PD2-Typ-MS -> Inductor_SMD:L_Wuerth_WE-TPC-3816
Connections:
- net BAT_IN is gone; now on net +7.5V: D4.2 (A), R6.2
- net +3.3V: now also J3.2 (Pin_2), J4.2 (Pin_2), J7.2 (Pin_2); no longer J3.3 (Pin_3), J4.3 (Pin_3)
- net BAT_OUT: no longer J7.2 (Pin_2)
- net ESP32-IR-FL: now also J3.3 (Pin_3); no longer J3.2 (Pin_2)
- net ESP32-IR-FR: now also J4.3 (Pin_3); no longer J4.2 (Pin_2)
- net ESP32-SRV-F: no longer J7.1 (Pin_1)
- net ESP32-LF-RIGHT: now reaches U2.5 (GPIO5/TOUCH5/ADC1_CH4)
- net ESP32-LF-LEFT: now reaches U2.6 (GPIO6/TOUCH6/ADC1_CH5)
- net ESP32-REMOTE: now reaches U2.7 (GPIO7/TOUCH7/ADC1_CH6)
- net ESP32-REMOTE: now also J7.1 (Pin_1)
- no-connect marks 33 -> 30
Other:
- note added: "The connectors should follow below modules: LF: (out, +, -) https://www.aliexpress.com/item/1005005643822767.html?spm=a2g0o.productlist.main.3.341c794f4rmnMT&algo_pvid=a06fe814-6544-4f6f-84ae-744686a22781&algo_exp_id=a06fe814-6544-4f6f-84ae-744686a22781-1&pdp_npi=4%40dis%21EUR%211.27%210.82%21%21%219.68%216.29%21%402103956b17063697430184239ebd04%2112000033861011923%21sea%21SE%21939121189%21&curPa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"
- note removed: "power switch before the buck converter, close to the battery."
- moved on the sheet: C11, C4, C5, C9, J10, L1, U3
