File: board/bubblebutbot/bubblebutbot.kicad_pcb (KiCad board)
At the start: 2 copper layers, 90 x 30 mm, 69 parts, among them J1 JST XH, J10 JST XH, J11 JST XH, J13 JST XH, J2 USB_C_Receptacle, J3 Conn_01x03_Socket, J4 Conn_01x03_Socket, J5 Conn_01x03_Socket, J6 Conn_01x03_Socket, J7 Conn_01x03_Socket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

Commit message: pcb 1v04
Parts:
- removed BZ1: Buzzer, Buzzer_Beeper:MagneticBuzzer_PUI_AT-0927-TT-6-R
- removed J8: Conn_01x03_Socket, Connector_JST:JST_PH_S3B-PH-K_1x03_P2.00mm_Horizontal
- removed R13: 5.1K, Resistor_SMD:R_0603_1608Metric_Pad0.98x0.95mm_HandSolder
- removed boot, rst: SW_Push, Button_Switch_SMD:SW_SPST_B3U-1000P
- removed kibuzzard-6507382A: G***, kibuzzard-6507382A
- removed kibuzzard-6507384E: G***, kibuzzard-6507384E
- removed kibuzzard-6507385B: G***, kibuzzard-6507385B
- added C13: 1u, Capacitor_SMD:C_0603_1608Metric_Pad1.08x0.95mm_HandSolder, F.Cu at (110.7, 46.6)
- added C14: 0.1uF/50V, Capacitor_SMD:C_0603_1608Metric_Pad1.08x0.95mm_HandSolder, F.Cu at (88.8, 31.9)
- added C16: 22u, Capacitor_SMD:C_1206_3216Metric_Pad1.33x1.80mm_HandSolder, F.Cu at (75.5, 50.9)
- added D4: SS14, Diode_SMD:D_SMA, F.Cu at (77.8, 40.7)
- added R3: 100k, Resistor_SMD:R_0603_1608Metric_Pad0.98x0.95mm_HandSolder, F.Cu at (81.2, 52.0)
- added SW1: SW_Push, Button_Switch_SMD:SW_SPST_CK_RS282G05A3, F.Cu at (113.8, 41.1)
- added SW2: SW_Push, Button_Switch_SMD:SW_SPST_CK_RS282G05A3, F.Cu at (118.4, 41.1)
- added U2: ESP32-S3-WROOM-1, RF_Module:ESP32-S3-WROOM-1, F.Cu at (97.8, 47.4)
- added kibuzzard-65510192: G***, kibuzzard-65510192, F.Cu at (118.5, 46.7)
- added kibuzzard-655101A0: G***, kibuzzard-655101A0, F.Cu at (113.9, 46.7)
- C11: value 100n -> 10n
- C3: value 10u -> 0.1uF/50V
- J5, J6: value Conn_01x03_Socket -> Conn_01x01_Pin; footprint Connector_JST:JST_PH_S3B-PH-K_1x03_P2.00mm_Horizontal -> TestPoint:TestPoint_Pad_2.0x2.0mm
- R11: value 50k -> 100k
- R16: value R -> 12k
- U5: value ~ -> SY8303
- kibuzzard-650738AB: moved to B.Cu
- moved J6 68.9 mm to (72.2, 42.8)
- moved kibuzzard-650738AB 65.4 mm to (71.5, 51.0), turned to 180 degrees
- moved J5 53.6 mm to (68.6, 42.8)
- moved H2 20.0 mm to (116.1, 50.5)
- moved C3 14.6 mm to (108.8, 46.6), turned to 90 degrees
- moved R1 13.0 mm to (109.7, 49.3), turned to 180 degrees
- moved kibuzzard-65073881 12.4 mm to (141.4, 37.3)
- moved J9 12.4 mm to (140.4, 39.9)
- moved kibuzzard-65073819 11.7 mm to (124.7, 37.3)
- moved J11 11.6 mm to (123.7, 39.9)
- moved kibuzzard-65073803 10.2 mm to (141.3, 34.5)
- moved J13 10.1 mm to (142.4, 31.9)
- moved J4 9.94 mm to (135.1, 31.9)
- moved kibuzzard-650737FA 9.94 mm to (133.1, 34.5)
- moved J7 9.84 mm to (131.1, 39.9), turned to 0 degrees
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Connections:
- C12 pad 1: 5V_BAT -> Net-(D4-A)
- C9 pad 1: +7.5V -> BAT_OUT
- J5 pad 1: GND -> +7.5V
- J6 pad 1: GND -> BAT_OUT
- J7 pad 1: GND -> ESP32-SRV-F
- J7 pad 2: ESP32-SRV-F -> +5V
- J7 pad 3: +5V -> GND
- L1 pad 2: 5V_BAT -> Net-(D4-A)
- R11 pad 1: +5V -> Net-(U1-nSLEEP)
- R11 pad 2: Net-(U1-nSLEEP) -> +5V
- R15 pad 2: 5V_BAT -> Net-(D4-A)
- R6 pad 2: +7.5V -> BAT_OUT
- U2 pad 10: ESP32-SRV-B -> ESP32-SRV-F
- U2 pad 11: ESP32-SRV-F -> ESP32-IR-FR
- U2 pad 12: unconnected-(U2-GPIO8/TOUCH8/ADC1_CH7/SUBSPICS1-Pad12) -> ESP32-IR-FL
- U2 pad 38: ESP32-BUZZER -> unconnected-(U2-GPIO2/TOUCH2/ADC1_CH1-Pad38)
- U2 pad 4: ESP32-IR-BR -> unconnected-(U2-GPIO4/TOUCH4/ADC1_CH3-Pad4)
- U2 pad 5: ESP32-IR-BL -> unconnected-(U2-GPIO5/TOUCH5/ADC1_CH4-Pad5)
- U2 pad 6: ESP32-IR-FR -> unconnected-(U2-GPIO6/TOUCH6/ADC1_CH5-Pad6)
- U2 pad 7: ESP32-IR-FL -> unconnected-(U2-GPIO7/TOUCH7/ADC1_CH6-Pad7)
- U5 pad 5: +7.5V -> BAT_OUT
Routing:
- net ESP32-BUZZER: track 70.4 -> 0.00 mm, vias 1 -> 0
- net ESP32-IR-BR: track 38.9 -> 0.00 mm, vias 2 -> 0
- net ESP32-SRV-B: track 30.0 -> 0.00 mm, vias 1 -> 0
- net BAT_OUT: track 0.00 -> 24.0 mm
- net +5V: track 97.7 -> 78.0 mm
- net ESP32-IR-BL: track 19.6 -> 0.00 mm
- net MOTOR-RIGHT-BR: track 60.7 -> 41.0 mm
- net ESP32-RESET: track 25.1 -> 10.5 mm, vias 2 -> 0
- net MOTOR-RIGHT-BL: track 61.0 -> 46.5 mm
- net +3.3V: track 45.9 -> 32.7 mm, vias 7 -> 5
- net ESP32-IR-FR: track 42.6 -> 31.7 mm, vias 0 -> 1
- net ESP32-BATTERY-READ: track 10.7 -> 5.71 mm
- net MOTOR-LEFT-BR: track 25.8 -> 21.2 mm, vias 2 -> 0
- net MOTOR-LEFT-BL: track 23.7 -> 19.5 mm, vias 2 -> 0
- net ESP32-SRV-F: track 31.2 -> 27.3 mm, vias 1 -> 0
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- added copper zone on F.Cu, net Net-(D4-A)
- removed copper zone on F.Cu, net +7.5V
- removed copper zone on F.Cu, net Net-(U5-FB)
Other:
- board size 90 x 30 mm -> 79.7 x 28.4 mm

Commit message: small fix
Routing:
- net +5V: track 78.0 -> 77.4 mm
Changed lines of the file:
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@@
     (fp_line (start 1.6 0.8) (end -1.6 0.8)
       (stroke (width 0.1) (type solid)) (layer "F.Fab"))
-    (pad "1" smd roundrect locked (at -1.5625 0 270) (size 1.325 1.8) (layers "F.Cu" "F.Paste" "F.Mask") (roundrect_rratio 0.188679)
+    (pad "1" smd roundrect locked (at -1.5625 0 270) (size 1.325 1.8) (layers "F.Cu" "F.Paste" "F.Mask") (roundrect_rratio 0.1886792453)
       (net 1 "BAT_OUT") (pintype "passive"))
-    (pad "2" smd roundrect locked (at 1.5625 0 270) (size 1.325 1.8) (layers "F.Cu" "F.Paste" "F.Mask") (roundrect_rratio 0.188679)
+    (pad "2" smd roundrect locked (at 1.5625 0 270) (size 1.325 1.8) (layers "F.Cu" "F.Paste" "F.Mask") (roundrect_rratio 0.1886792453)
       (net 2 "GND") (pintype "passive"))
     (model "${KICAD6_3DMODEL_DIR}/Capacitor_SMD.3dshapes/C_1206_3216Metric.wrl"
@@
   (segment (start 110.175 32.625) (end 112.4 30.4) (width 0.5) (layer "B.Cu") (net 5))
   (segment (start 131.1 36.3) (end 133.1 38.3) (width 0.5) (layer "B.Cu") (net 5))
-  (segment (start 105.084314 35.784314) (end 105.468629 35.4) (width 0.5) (layer "B.Cu") (net 5))
   (segment locked (start 85.6 37.8) (end 85.6 35.8) (width 0.5) (layer "B.Cu") (net 5))
   (segment (start 112.4 30.4) (end 120.7 30.4) (width 0.5) (layer "B.Cu") (net 5))

Commit message: pcb v0.5
smaller
Parts:
- removed J11, J9: JST XH, Connector_JST:JST_PH_S2B-PH-K_1x02_P2.00mm_Horizontal
- removed kibuzzard-65073819: G***, kibuzzard-65073819
- removed kibuzzard-65073881: G***, kibuzzard-65073881
- removed kibuzzard-650738AB: G***, kibuzzard-650738AB
- added kibuzzard-656B6852: G***, kibuzzard-656B6852, B.Cu at (97.7, 48.9)
- added kibuzzard-656B6902: G***, kibuzzard-656B6902, B.Cu at (101.6, 50.5)
- added kibuzzard-656B692B: G***, kibuzzard-656B692B, B.Cu at (101.1, 51.8)
- added kibuzzard-656B6B05: G***, kibuzzard-656B6B05, F.Cu at (97.3, 27.6)
- added kibuzzard-656B6B82: G***, kibuzzard-656B6B82, F.Cu at (112.1, 50.2)
- added kibuzzard-656B6B9B: G***, kibuzzard-656B6B9B, F.Cu at (87.3, 36.8)
- added kibuzzard-656B6BB3: G***, kibuzzard-656B6BB3, F.Cu at (87.4, 51.3)
- moved J13 20.2 mm to (123.8, 39.9), turned to 0 degrees
- moved kibuzzard-65073803 16.7 mm to (124.8, 37.3)
- moved J7 0.10 mm to (131.1, 40.0)
- turned SW2 to 90 degrees
Connections:
- net MOTOR-LEFT-BL renamed MOTOR-LEFT-FL
- net MOTOR-LEFT-BR renamed MOTOR-LEFT-FR
- net MOTOR-RIGHT-BL renamed MOTOR-RIGHT-FL
- net MOTOR-RIGHT-BR renamed MOTOR-RIGHT-FR
Routing:
- net MOTOR-RIGHT-FL: track 46.5 -> 17.6 mm, vias 0 -> 1
- net MOTOR-RIGHT-FR: track 41.0 -> 19.4 mm, vias 0 -> 1
- net MOTOR-LEFT-FR: track 21.2 -> 5.33 mm
- net MOTOR-LEFT-FL: track 19.5 -> 7.86 mm
- net ESP32-BOOT0: track 41.0 -> 39.4 mm
- net GND: vias 80 -> 72
Other:
- board size 79.7 x 28.4 mm -> 72.2 x 28.4 mm
- board text added: "a) Search for the {dblquote}BattleButBot{dblquote} Wi-Fi network b) Connect c) Open your browser d) Type {dblquote}bot.local{dblquote} as the URL e) ? f) Enjoy :)"

Commit message: Working on the new version ... 🚀
Parts:
- removed C12: 22u, Capacitor_SMD:C_1206_3216Metric_Pad1.33x1.80mm_HandSolder
- removed Q1: FDN336P, Package_TO_SOT_SMD:SOT-23
- removed R10: 5.1K, Resistor_SMD:R_0603_1608Metric_Pad0.98x0.95mm_HandSolder
- removed R14, R15, R3, R8: 100k, Resistor_SMD:R_0603_1608Metric_Pad0.98x0.95mm_HandSolder
- removed R16: 12k, Resistor_SMD:R_0603_1608Metric_Pad0.98x0.95mm_HandSolder
- removed U5: SY8303, Package_TO_SOT_SMD:SOT-23-8
- C11: value 10n -> 100n
- C4, C5: value 1u -> 22u; footprint Capacitor_SMD:C_0603_1608Metric_Pad1.08x0.95mm_HandSolder -> Capacitor_SMD:C_1206_3216Metric_Pad1.33x1.80mm_HandSolder
- L1: value 4.7u -> 3.3u; footprint Inductor_SMD:L_Wuerth_WE-TPC-3816 -> Inductor_SMD:L_Wuerth_WE-PD2-Typ-MS
- U3: value AP2112K-3.3 -> AP63203WU; footprint Package_TO_SOT_SMD:SOT-23-5 -> Package_TO_SOT_SMD:TSOT-23-6
- moved L1 32.7 mm to (46.0, 34.5)
- moved C4 31.2 mm to (57.5, 31.4)
- moved C11 31.1 mm to (53.0, 35.5)
- moved U3 30.7 mm to (56.6, 38.5)
- moved C5 28.8 mm to (53.5, 31.5)
- moved D4 28.8 mm to (49.0, 42.0)
- moved D2 27.4 mm to (59.0, 45.0)
- moved C9 22.7 mm to (58.5, 50.2)
- moved C16 2.62 mm to (74.5, 48.5)
Connections:
- C11 pad 1: Net-(U5-BS) -> Net-(U3-SW)
- C11 pad 2: Net-(U5-LX) -> Net-(U3-BST)
- C16 pad 1: BAT_OUT -> BAT_IN
- C5 pad 1: +5V -> +3.3V
- C8 pad 2: +5V -> BAT_OUT
- C9 pad 2: Net-(U5-EN) -> GND
- D2 pad 1: +5V -> BAT_OUT
- D4 pad 1: 5V_BAT -> BAT_OUT
- D4 pad 2: Net-(D4-A) -> BAT_IN
- J3 pad 3: +5V -> +3.3V
- J4 pad 3: +5V -> +3.3V
- J6 pad 1: BAT_OUT -> BAT_IN
- J7 pad 2: +5V -> BAT_OUT
- L1 pad 1: Net-(U5-LX) -> Net-(U3-SW)
- L1 pad 2: Net-(D4-A) -> +3.3V
- R11 pad 2: +5V -> BAT_OUT
- R6 pad 2: BAT_OUT -> BAT_IN
- U1 pad 12: +5V -> BAT_OUT
- U3 pad 1: +5V -> +3.3V
- U3 pad 2: GND -> BAT_OUT
- U3 pad 3: Net-(U3-EN) -> BAT_OUT
- U3 pad 4: unconnected-(U3-NC-Pad4) -> GND
- U3 pad 5: +3.3V -> Net-(U3-SW)
Routing:
- net +5V: track 77.4 -> 0.00 mm, vias 5 -> 0
- net BAT_OUT: track 24.0 -> 42.2 mm, vias 0 -> 2
- net 5V_USB_POWER: track 20.3 -> 6.53 mm
- net Net-(U5-EN): track 6.14 -> 0.00 mm
- net ESP32-BATTERY-READ: track 5.71 -> 0.00 mm
- net Net-(U5-FS): track 5.58 -> 0.00 mm
- net Net-(U5-FB): track 3.79 -> 0.00 mm
- net Net-(U5-BS): track 2.24 -> 0.00 mm
- net Net-(U3-EN): track 1.84 -> 0.00 mm
- net GND: vias 72 -> 71
- removed copper zone on F.Cu, net +5V
- removed copper zone on F.Cu, net 5V_BAT
- removed copper zone on F.Cu, net 5V_USB_POWER
- removed copper zone on F.Cu, net Net-(D4-A)
- removed copper zone on F.Cu, net Net-(U5-LX)

Commit message: VERSION 1.06
Parts:
- removed C16: 22u, Capacitor_SMD:C_1206_3216Metric_Pad1.33x1.80mm_HandSolder
- removed J5, J6: Conn_01x01_Pin, TestPoint:TestPoint_Pad_2.0x2.0mm
- removed kibuzzard-6507374A: G***, kibuzzard-6507374A
- removed kibuzzard-6507377B: G***, kibuzzard-6507377B
- removed kibuzzard-65073792: G***, kibuzzard-65073792
- removed kibuzzard-650737FA: G***, kibuzzard-650737FA
- removed kibuzzard-65073803: G***, kibuzzard-65073803
- removed kibuzzard-650739D2: G***, kibuzzard-650739D2
- removed kibuzzard-650739DD: G***, kibuzzard-650739DD
- removed kibuzzard-650739F6: G***, kibuzzard-650739F6
- removed kibuzzard-65510192: G***, kibuzzard-65510192
- removed kibuzzard-655101A0: G***, kibuzzard-655101A0
- removed kibuzzard-656B6852: G***, kibuzzard-656B6852
- removed kibuzzard-656B6902: G***, kibuzzard-656B6902
- removed kibuzzard-656B692B: G***, kibuzzard-656B692B
- removed kibuzzard-656B6B05: G***, kibuzzard-656B6B05
- removed kibuzzard-656B6B82: G***, kibuzzard-656B6B82
- removed kibuzzard-656B6B9B: G***, kibuzzard-656B6B9B
- added kibuzzard-65B52192: G***, kibuzzard-65B52192, F.Cu at (68.4, 26.8)
- added kibuzzard-65B521AC: G***, kibuzzard-65B521AC, F.Cu at (97.1, 27.9)
- added kibuzzard-65B53096: G***, kibuzzard-65B53096, F.Cu at (74.5, 52.5)
- added kibuzzard-65B53492: G***, kibuzzard-65B53492, F.Cu at (133.1, 37.3)
- added kibuzzard-65B534AD: G***, kibuzzard-65B534AD, F.Cu at (124.8, 37.3)
- added kibuzzard-65B534B8: G***, kibuzzard-65B534B8, F.Cu at (115.5, 34.6)
- added kibuzzard-65B534D1: G***, kibuzzard-65B534D1, F.Cu at (123.8, 34.6)
- added kibuzzard-65B534EC: G***, kibuzzard-65B534EC, F.Cu at (133.1, 34.6)
- added kibuzzard-65B53575: G***, kibuzzard-65B53575, F.Cu at (113.9, 46.9)
- added kibuzzard-65B5357F: G***, kibuzzard-65B5357F, F.Cu at (118.4, 46.9)
- added kibuzzard-65B53DEB: G***, kibuzzard-65B53DEB, F.Cu at (83.2, 52.0)
- added kibuzzard-65B53F64: G***, kibuzzard-65B53F64, B.Cu at (108.4, 39.5)
- added kibuzzard-65B53FA4: G***, kibuzzard-65B53FA4, B.Cu at (104.2, 37.6)
- added kibuzzard-65B5507C: G***, kibuzzard-65B5507C, B.Cu at (107.1, 41.2)
- L1: footprint Inductor_SMD:L_Wuerth_WE-PD2-Typ-MS -> Inductor_SMD:L_Wuerth_WE-TPC-3816
- moved L1 39.8 mm to (85.4, 28.8), turned to 90 degrees
- moved D4 36.5 mm to (85.4, 40.0), turned to -90 degrees
- moved C5 31.8 mm to (85.3, 32.5), turned to 180 degrees
- moved C11 29.4 mm to (81.0, 26.8)
- moved C9 28.3 mm to (80.3, 32.1)
- moved C4 28.0 mm to (85.3, 35.0), turned to 180 degrees
- moved U3 25.7 mm to (80.7, 29.4)
- moved D2 23.2 mm to (81.7, 40.0), turned to -90 degrees
- moved R4 11.6 mm to (72.3, 47.4)
- moved R7 10.6 mm to (74.0, 47.4)
- moved J1 9.59 mm to (77.8, 47.6)
- moved D3 7.51 mm to (73.2, 33.6)
- moved J2 7.34 mm to (74.9, 39.9)
- moved R17 7.28 mm to (76.7, 33.6)
- moved R6 5.55 mm to (84.2, 46.5)
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Connections:
- D4 pad 2: BAT_IN -> +7.5V
- J3 pad 2: ESP32-IR-FL -> +3.3V
- J3 pad 3: +3.3V -> ESP32-IR-FL
- J4 pad 2: ESP32-IR-FR -> +3.3V
- J4 pad 3: +3.3V -> ESP32-IR-FR
- J7 pad 1: ESP32-SRV-F -> ESP32-REMOTE
- J7 pad 2: BAT_OUT -> +3.3V
- R6 pad 2: BAT_IN -> +7.5V
- U2 pad 5: unconnected-(U2-GPIO5/TOUCH5/ADC1_CH4-Pad5) -> ESP32-LF-RIGHT (x2)
- U2 pad 6: unconnected-(U2-GPIO6/TOUCH6/ADC1_CH5-Pad6) -> ESP32-LF-LEFT (x2)
- U2 pad 7: unconnected-(U2-GPIO7/TOUCH7/ADC1_CH6-Pad7) -> ESP32-REMOTE (x2)
Routing:
- net +3.3V: track 32.7 -> 89.9 mm, vias 5 -> 9
- net ESP32-SRV-F: track 27.3 -> 0.00 mm
- net ESP32-REMOTE: track 0.00 -> 26.7 mm
- net ESP32-BATTERY-READ: track 0.00 -> 7.63 mm
- net ESP32-D-: track 41.9 -> 34.3 mm
- net ESP32-D+: track 46.8 -> 39.3 mm
- net Net-(J2-CC1): track 4.96 -> 11.2 mm
- net Net-(J2-CC2): track 2.68 -> 7.27 mm
- net ESP32-IR-FR: track 31.7 -> 27.9 mm, vias 1 -> 0
- net +7.5V: track 5.53 -> 9.32 mm
- net 5V_USB_POWER: track 6.53 -> 9.43 mm
- net Net-(U3-BST): track 0.00 -> 2.37 mm
- net ESP32-IR-FL: track 21.2 -> 20.3 mm, vias 1 -> 0
- net ESP32-BOOT0: track 39.4 -> 38.8 mm
- net BAT_OUT: track 42.2 -> 41.7 mm, vias 2 -> 3
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- added copper zone on F.Cu, net BAT_OUT
- added copper zone on F.Cu, net Net-(U3-SW)
Other:
- board size 72.2 x 28.4 mm -> 66.5 x 28.4 mm
